Commit message: imu/encoder/ekf ready

File: jetson/robot_ws/src/robot_navigation/urdf/base/summit_base.urdf (robot description, URDF)
Before this commit: robot mecanum_robot, 7 links, 6 joints
Links:
- added link imu_link, mass 0.001; visual box size=0.01 0.01 0.01
Joints:
- added joint imu_joint: type fixed, parent base_link, child imu_link, origin xyz=0 0 0.03 rpy=0 0 0
