Commit message: Logs e testes navegação

File: jetson/robot_ws/src/robot_description/urdf/robot_description.urdf (robot description, URDF)
Before this commit: robot robot_description, 8 links, 7 joints
Joints:
- joint pulso_joint: origin xyz=0.325 0 0.07557 rpy=-3.1416 0 0 -> xyz=0.325 0 0.07557 rpy=-3.1416 0 3.14159

Commit message: final_urdf

File: jetson/robot_ws/src/robot_description/urdf/robot_description.urdf (robot description, URDF)
Before this commit: robot robot_description, 8 links, 7 joints
Links:
- added link base_footprint
- link base_link: mass 3.8406 -> 3.6752
Joints:
- added joint base_link_joint: type fixed, parent base_footprint, child base_link, origin xyz=0 0 0 rpy=0 0 3.1416

Commit message: last_changes

File: jetson/robot_ws/src/robot_description/urdf/robot_description.urdf (robot description, URDF)
Before this commit: robot robot_description, 9 links, 8 joints
Links:
- removed link base_footprint
- removed link lidar_link
- removed link realsense_link
- added link camera_link, mass 0.087339; collision mesh filename=package://robot_description/meshes/realsense_link.STL; visual mesh filename=package://robot_description/meshes/realsense_link.STL
- added link laser, mass 0.16538; collision mesh filename=package://robot_description/meshes/lidar_link.STL; visual mesh filename=package://robot_description/meshes/lidar_link.STL
Joints:
- removed joint base_link_joint
- removed joint realsense_joint
- added joint camera_joint: type fixed, parent base_link, child camera_link, origin xyz=0.072916 0 -0.058189 rpy=0 0.17453 0, axis 0 0 0
- joint lidar_joint: child lidar_link -> laser; origin xyz=0.036445 0 -0.124 rpy=0 0 0 -> xyz=0.036445 0 -0.124 rpy=0 0 1.57

Commit message: att navigation

File: jetson/robot_ws/src/robot_description/urdf/robot_description.urdf (robot description, URDF)
Before this commit: robot robot_description, 9 links, 8 joints
Links:
- removed link lidar_link
- removed link realsense_link
- added link camera_link, mass 0.087339; collision mesh filename=package://robot_description/meshes/realsense_link.STL; visual mesh filename=package://robot_description/meshes/realsense_link.STL
- added link laser, mass 0.16538; collision mesh filename=package://robot_description/meshes/lidar_link.STL; visual mesh filename=package://robot_description/meshes/lidar_link.STL
Joints:
- removed joint lidar_joint
- removed joint realsense_joint
- added joint camera_joint: type fixed, parent base_link, child camera_link, origin xyz=0.072916 0 -0.058189 rpy=0 0.17453 0, axis 0 0 0
- added joint laser_joint: type fixed, parent base_link, child laser, origin xyz=0.036445 0 -0.124 rpy=0 0 -1.57, axis 0 0 0

File: jetson/robot_ws/src/robot_description/urdf/robot_description_sim.urdf (robot description, URDF)
Before this commit: robot robot_description, 10 links, 9 joints
Joints:
- joint lidar_joint: origin xyz=0 0 0.1 rpy=0 0 0 -> xyz=0.036445 0 -0.124 rpy=0 0 0

Commit message: URDF atual do robô atualizado

File: jetson/robot_ws/src/robot_description/urdf/robot_description.urdf (robot description, URDF)
Before this commit: robot robot_description, 9 links, 8 joints
Links:
- removed link base_footprint
Joints:
- removed joint base_link_joint
- removed joint laser_joint
- added joint lidar_joint: type fixed, parent base_link, child laser, origin xyz=0.036445 0 -0.124 rpy=0 0 1.57, axis 0 0 0
- joint pulso_joint: origin xyz=0.325 0 0.07557 rpy=-3.1416 0 0 -> xyz=0.325 0 0.07557 rpy=-3.1416 0 3.14159

File: jetson/robot_ws/src/robot_description/urdf/robot_description_sim.urdf (robot description, URDF)
Before this commit: robot robot_description, 10 links, 9 joints
Links:
- removed link base_footprint
- removed link imu_link
- removed link lidar_link
- removed link realsense_link
- added link camera_link, mass 0.087339; collision mesh filename=package://robot_description/meshes/realsense_link.STL; visual mesh filename=package://robot_description/meshes/realsense_link.STL
- added link laser, mass 0.16538; collision mesh filename=package://robot_description/meshes/lidar_link.STL; visual mesh filename=package://robot_description/meshes/lidar_link.STL
- link base_link: mass 3.8406 -> 3.6752
Joints:
- removed joint base_link_joint
- removed joint imu_joint
- removed joint realsense_joint
- added joint camera_joint: type fixed, parent base_link, child camera_link, origin xyz=0.072916 0 -0.058189 rpy=0 0.17453 0, axis 0 0 0
- joint lidar_joint: axis (none) -> 0 0 0; child lidar_link -> laser; origin xyz=0.036445 0 -0.124 rpy=0 0 0 -> xyz=0.036445 0 -0.124 rpy=0 0 1.57
- joint pulso_joint: origin xyz=0.325 0 0.07557 rpy=-3.1416 0 0 -> xyz=0.325 0 0.07557 rpy=-3.1416 0 3.14159

Commit message: mapping corrected

File: jetson/robot_ws/src/robot_description/urdf/robot_description.urdf (robot description, URDF)
Before this commit: robot robot_description, 8 links, 7 joints
Joints:
- joint lidar_joint: origin xyz=0.036445 0 -0.124 rpy=0 0 1.57 -> xyz=0.036445 0 -0.124 rpy=0 3.14159 1.57

File: jetson/robot_ws/src/robot_description/urdf/robot_description_sim.urdf (robot description, URDF)
Before this commit: robot robot_description, 10 links, 9 joints
Links:
- removed link garra1_link
- removed link garra2_link
- removed link imu_link
- removed link lidar_link
- removed link manip_link
- removed link plat_link
- removed link pulso_link
- removed link realsense_link
- added link camera_link, mass 0.001; visual box size=0.01 0.01 0.01
- added link laser, mass 1.0; collision cylinder length=0.0125 radius=0.0125; visual cylinder length=0.0125 radius=0.0125
- added link wheel_front_left, mass 2.0; collision cylinder length=0.0125 radius=0.025; visual cylinder length=0.0125 radius=0.025
- added link wheel_front_right, mass 2.0; collision cylinder length=0.0125 radius=0.025; visual cylinder length=0.0125 radius=0.025
- added link wheel_rear_left, mass 2.0; collision cylinder length=0.0125 radius=0.025; visual cylinder length=0.0125 radius=0.025
- added link wheel_rear_right, mass 2.0; collision cylinder length=0.0125 radius=0.025; visual cylinder length=0.0125 radius=0.025
- link base_footprint: geometry visual box size=0.00025 0.00025 0.00025
- link base_link: mass 3.8406 -> 50.0; geometry collision box size=0.15 0.15 0.025; visual box size=0.15 0.15 0.025
Joints:
- removed joint garra1_joint
- removed joint garra2_joint
- removed joint imu_joint
- removed joint lidar_joint
- removed joint manip_joint
- removed joint plat_joint
- removed joint pulso_joint
- removed joint realsense_joint
- added joint camera_joint: type fixed, parent base_link, child camera_link, origin xyz=0.072916 0 0 rpy=0 0.17453 0
- added joint joint_wheel_front_left: type revolute, parent base_link, child wheel_front_left, origin xyz=0.075 0.075 0.0125 rpy=0 0 0, axis 0 1 0, limit effort=100 velocity=10
- added joint joint_wheel_front_right: type revolute, parent base_link, child wheel_front_right, origin xyz=0.075 -0.075 0.0125 rpy=0 0 0, axis 0 1 0, limit effort=100 velocity=10
- added joint joint_wheel_rear_left: type revolute, parent base_link, child wheel_rear_left, origin xyz=-0.075 0.075 0.0125 rpy=0 0 0, axis 0 1 0, limit effort=100 velocity=10
- added joint joint_wheel_rear_right: type revolute, parent base_link, child wheel_rear_right, origin xyz=-0.075 -0.075 0.0125 rpy=0 0 0, axis 0 1 0, limit effort=100 velocity=10
- added joint laser_joint: type fixed, parent base_link, child laser, origin xyz=0.036445 0 0.13 rpy=0 0 -1.57
- joint base_link_joint: origin xyz=0 0 0 rpy=0 0 3.1416 -> xyz=0 0 0.0125 rpy=0 0 0
